File: pcb/v1/hobgoblin_v1.sch (KiCad schematic (older format))
At the start: 45 parts, among them J1 5V, J2 RC2014EXT1, J3 RC2014EXT2, SW1 RESET, SW2 ROMBNK, U1 74LS32, U2 Z80CPU, U3 74LS14, U4 74LS138, U5 628128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

Commit message: Fix IOWR/IORD pins on CF socket
Parts:
- added unit 2 of U1
Connections:
- net ~IORQ: now also U1.4
- net ~IOWR: now also CF1.35 (~IOWR)
- net ~RD: now also U1.5; no longer CF1.34 (~IORD)
- net ~WR: no longer CF1.35 (~IOWR)
- new net ~IORD: CF1.34 (~IORD), U1.6
Changed lines of the file:
@@
 NoConn ~ 9150 1700
 Text Label 9150 2600 0    50   ~ 0
-~RD
+~IORD
 Text Label 9150 2500 0    50   ~ 0
-~WR
+~IOWR
 NoConn ~ 9150 2300
 $Comp
@@
 	1    0    0    -1
 $EndComp
+$Comp
+L 74xx:74LS32 U1
+U 2 1 600D80CC
+P 1100 4950
+F 0 "U1" H 1100 4950 50  0000 C CNN
+F 1 "74LS32" H 1300 5100 50  0000 C CNN
+F 2 "" H 1100 4950 50  0001 C CNN
+F 3 "http://www.ti.com/lit/gpn/sn74LS32" H 1100 4950 50  0001 C CNN
+	2    1100 4950
+	1    0    0    -1
+$EndComp
+Text Label 1400 4950 0    50   ~ 0
+~IORD
+Text Label 800  4850 2    50   ~ 0
+~IORQ
+Text Label 700  5050 2    50   ~ 0
+~RD
+Wire Wire Line
+	700  5050 800  5050
 $EndSCHEMATC

Commit message: Final 1.3 routing improvements
Connections:
- net VCC: no longer U4.6 (E3)
- net ~M1: now also U4.6 (E3)
Changed lines of the file:
@@
 Text Label 2000 5100 0    50   ~ 0
 A5
-$Comp
-L power:VCC #PWR011
-U 1 1 5FBC9D21
-P 2100 5400
-F 0 "#PWR011" H 2100 5250 50  0001 C CNN
-F 1 "VCC" H 2115 5573 50  0000 C CNN
-F 2 "" H 2100 5400 50  0001 C CNN
-F 3 "" H 2100 5400 50  0001 C CNN
-	1    2100 5400
-	1    0    0    -1
-$EndComp
 Wire Wire Line
 	2000 5500 2100 5500
@@
 Wire Wire Line
 	700  5050 800  5050
+Text Label 2100 5400 2    50   ~ 0
+~M1
 $EndSCHEMATC
