File: pcb/v2/USB_UART.kicad_sch (KiCad schematic)
At the start: 0 parts

Commit message: Draft component placement
Parts:
- added C14: 10uF, Capacitor_THT:CP_Radial_D4.0mm_P1.50mm, symbol Device:C
- added C15, C16: 0.1uF, Capacitor_THT:C_Disc_D3.8mm_W2.6mm_P2.50mm, symbol Device:C
- added J4: MINIUSB, Connector_USB:USB_Mini-B_Lumberg_2486_01_Horizontal, symbol hobgoblin_v1-rescue:USB_B_Mini-Connector
- added JP1: USB_VCC, Connector_PinSocket_2.54mm:PinSocket_1x02_P2.54mm_Vertical, symbol Jumper:Jumper_2_Bridged
- added U5: FT232RL, Package_SO:SSOP-28_5.3x10.2mm_P0.65mm, symbol Interface_USB:FT232RL
Connections:
- new net: J4.1 (VBUS), JP1.1 (A)
- new net: C15.2, U5.17 (3V3OUT)
- new net GND: C14.2, C15.1, C16.2, J4.5 (GND), J4.6 (Shield), U5.18 (GND), U5.21 (GND), U5.25 (AGND), U5.26 (TEST), U5.7 (GND)
- new net RX: U5.1 (TXD)
- new net TX: U5.5 (RXD)
- new net USBD+: J4.3 (D+), U5.15 (USBD+)
- new net USBD-: J4.2 (D-), U5.16 (USBD-)
- new net VCC: C14.1, C16.1, JP1.2 (B), U5.20 (VCC), U5.4 (VCCIO)
- new net ~{RTS}: U5.11 (CTS)
- no-connect marks 0 -> 14

Commit message: In-progress PCB layout
Connections:
- net USB_VCC: now reaches J4.1 (VBUS), JP1.1 (A)
Changed lines of the file:
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@@
     (stroke (width 0) (type default) (color 0 0 0 0))
+  )
+  (label "USB_VCC" (at 102.87 72.39 90)
+    (effects (font (size 1.27 1.27)) (justify left bottom))
   )
   (label "USBD-" (at 106.68 80.01 0)
