File: pcb/v2/hobgoblin_v2.kicad_pcb (KiCad board)
At the start: 2 copper layers, 160 x 120 mm, 56 parts, among them J1 5V, J2 RC2014EXT1, J3 RC2014EXT2, J4 MINIUSB, J5 USBUART, SW1 RESET, SW2 ROMBNK, U1 74LS32, U10 MC68B50, U2 74LS14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

Commit message: Made some progress in layout
Parts:
- moved R12 10.2 mm to (127.0, 131.0), turned to 0 degrees
- moved R8 3.00 mm to (123.0, 93.0)
- moved R9 3.00 mm to (123.0, 96.0)
- moved X1 2.06 mm to (58.5, 32.0)
- moved D3 1.80 mm to (133.5, 127.0)
Routing:
- net VCC: track 68.0 -> 374.1 mm, vias 0 -> 8
- net /TXD: track 28.0 -> 198.1 mm, vias 2 -> 4
- net /~{RTS}: track 0.00 -> 163.8 mm, vias 0 -> 2
- net /RXD: track 41.1 -> 196.6 mm, vias 2 -> 4
- net /D6: track 134.1 -> 277.4 mm, vias 4 -> 8
- net Net-(R1-Pad2): track 0.00 -> 94.7 mm, vias 0 -> 2
- net /~{INT}: track 30.2 -> 117.4 mm, vias 2 -> 4
- net /~{RESET}: track 15.0 -> 101.3 mm, vias 0 -> 4
- net /D4: track 217.2 -> 300.0 mm, vias 5 -> 6
- net /D7: track 186.0 -> 266.9 mm, vias 3 -> 5
- net /D3: track 214.2 -> 294.6 mm, vias 5 -> 7
- net /UART_CLK: track 0.00 -> 75.6 mm, vias 0 -> 1
- net /D5: track 204.6 -> 276.5 mm
- net /IORQ: track 0.00 -> 55.1 mm
- net /~{WR}: track 41.1 -> 85.4 mm, vias 0 -> 2
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
Commit message: Update to latest KiCAD version
Parts:
- removed REF1: hole1, MountingHole:MountingHole_3.2mm_M3_Pad
- removed REF1: hole3, MountingHole:MountingHole_3.2mm_M3_Pad
- removed REF1: hole4, MountingHole:MountingHole_3.2mm_M3_Pad
- removed REF1: hole2, MountingHole:MountingHole_3.2mm_M3_Pad
- added H1: hole1, MountingHole:MountingHole_3.2mm_M3, F.Cu at (23.5, 23.5)
- added H2: hole2, MountingHole:MountingHole_3.2mm_M3, F.Cu at (166.5, 23.5)
- added H3: hole3, MountingHole:MountingHole_3.2mm_M3, F.Cu at (23.5, 126.5)
- added H4: hole4, MountingHole:MountingHole_3.2mm_M3, F.Cu at (166.5, 126.5)
- moved C16 167.1 mm to (257.7, 22.1), turned to 0 degrees
- moved C5 154.6 mm to (186.8, 92.1), turned to 0 degrees
- moved C2 150.7 mm to (188.3, 130.3), turned to 0 degrees
- moved C6 139.5 mm to (186.8, 87.9), turned to 0 degrees
- moved C13 134.5 mm to (194.6, 117.1)
- moved C3 130.2 mm to (213.9, 93.7), turned to 0 degrees
- moved R1 129.0 mm to (192.5, 26.1)
- moved C7 125.3 mm to (254.2, 61.1), turned to 0 degrees
- moved C1 123.9 mm to (214.8, 98.6)
- moved R4 122.0 mm to (145.0, 125.5), turned to 180 degrees
- moved R3 119.2 mm to (200.9, 98.8)
- moved R5 117.8 mm to (145.0, 122.5), turned to 180 degrees
- moved SW2 115.0 mm to (152.5, 126.3), turned to 90 degrees
- moved R6 113.7 mm to (145.0, 119.5), turned to 180 degrees
- moved C4 103.4 mm to (254.2, 57.0), turned to 0 degrees
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Routing:
- net VCC: track 374.1 -> 0.00 mm, vias 8 -> 0
- net /D4: track 300.0 -> 0.00 mm, vias 6 -> 0
- net /D3: track 294.6 -> 0.00 mm, vias 7 -> 0
- net /D6: track 277.4 -> 0.00 mm, vias 8 -> 0
- net /D5: track 276.5 -> 0.00 mm, vias 5 -> 0
- net /D7: track 266.9 -> 0.00 mm, vias 5 -> 0
- net /A15: track 222.9 -> 0.00 mm, vias 6 -> 0
- net /A14: track 208.7 -> 0.00 mm, vias 6 -> 0
- net /TXD: track 198.1 -> 0.00 mm, vias 4 -> 0
- net /RXD: track 196.6 -> 0.00 mm, vias 4 -> 0
- net /A10: track 184.9 -> 0.00 mm, vias 4 -> 0
- net /A13: track 180.5 -> 0.00 mm, vias 4 -> 0
- net /A12: track 174.8 -> 0.00 mm, vias 4 -> 0
- net /A0: track 169.7 -> 0.00 mm, vias 2 -> 0
- net /~{RTS}: track 163.8 -> 0.00 mm, vias 2 -> 0
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- removed copper zone on B.Cu, net GND
- removed copper zone on F.Cu, net GND
Other:
- board size 160 x 120 mm -> 150 x 110 mm
- board text added: "150x110"
